File: KiCad Keyboard.kicad_pcb (KiCad board)
At the start: 2 copper layers, 93 parts, among them U1 TEENSY2.0

Commit message: Basic keyboard arrangement
Parts:
- moved D_M7 219.1 mm to (20.3, 118.1)
- moved D_M3 212.0 mm to (20.3, 80.0)
- moved D_M8 208.9 mm to (39.4, 118.1)
- moved D_M2 204.4 mm to (39.4, 61.0)
- moved D_M1 202.5 mm to (20.3, 61.0)
- moved D_M5 193.0 mm to (20.3, 99.1)
- moved D_M9 189.2 mm to (20.3, 137.2)
- moved D_M0 180.3 mm to (39.4, 137.2)
- moved D_Esc_0 180.2 mm to (69.8, 31.8)
- moved D_F1 172.6 mm to (88.9, 31.8)
- moved D_1 172.5 mm to (88.9, 59.7)
- moved D_Esc_1 171.7 mm to (77.5, 97.8)
- moved D_M4 171.3 mm to (39.4, 80.0)
- moved SW_M8 165.1 mm to (39.4, 116.8)
- moved SW_Esc_0 164.8 mm to (69.8, 30.5)
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
Commit message: Changing diodes to SMD
Parts:
- D_1, D_2, D_3, D_4, D_5, D_6, D_A1, D_B1, D_C1, D_D1, D_E1, D_Esc_0, D_Esc_1, D_F1, D_F2, D_F3, D_F4, D_F5, D_F6, D_F7, D_G1, D_Grave1, D_LAlt1, D_LCtrl1, D_LShift1, D_LSpace1, D_LSuper1, D_M0, D_M1, D_M2, D_M3, D_M4, D_M5, D_M6, D_M7, D_M8, D_M9, D_Q1, D_R1, D_S1, D_T1, D_Tab1, D_V1, D_W1, D_X1, D_Z1: footprint Stormboard_Keyboard:CHERRY_MX_DIODE -> Diodes_SMD:D_SMA_Standard
- moved D_6 63.3 mm to (245.3, 76.2), turned to 270 degrees
- moved D_LCtrl1 63.2 mm to (133.3, 152.4), turned to 270 degrees
- moved D_F6 63.1 mm to (245.3, 47.6), turned to 270 degrees
- moved D_Esc_1 62.8 mm to (138.1, 114.3), turned to 270 degrees
- moved D_LSuper1 62.8 mm to (157.2, 152.4), turned to 270 degrees
- moved D_T1 62.7 mm to (235.7, 95.2), turned to 270 degrees
- moved D_LShift1 62.5 mm to (142.9, 133.3), turned to 270 degrees
- moved D_LAlt1 62.5 mm to (181.0, 152.4), turned to 270 degrees
- moved D_F7 62.4 mm to (221.5, 114.3), turned to 270 degrees
- moved D_A1 62.4 mm to (164.3, 114.3), turned to 270 degrees
- moved D_D1 62.4 mm to (202.4, 114.3), turned to 270 degrees
- moved D_G1 62.4 mm to (240.5, 114.3), turned to 270 degrees
- moved D_S1 62.4 mm to (183.4, 114.3), turned to 270 degrees
- moved D_Z1 61.8 mm to (173.8, 133.3), turned to 270 degrees
- moved D_B1 61.8 mm to (250.0, 133.3), turned to 270 degrees
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Connections:
- U1 pad 10: /Column7 -> /Column5
- U1 pad 11: /Column2 -> /Column6
- U1 pad 12: /Column3 -> /Column7
- U1 pad 2: /Row0 -> /Row3
- U1 pad 3: /Row1 -> /Row2
- U1 pad 4: /Row2 -> /Row1
- U1 pad 5: /Row3 -> /Row0
- U1 pad 7: /Column4 -> /Column2
- U1 pad 8: /Column5 -> /Column3
- U1 pad 9: /Column6 -> /Column4
Other:
- board outline added: 202.4 x 138.1 mm
